File: MCU_Logger.kicad_sch (KiCad schematic)
At the start: 0 parts

Commit message: Added symbols to EEscheme
Parts:
- added BT1: Battery, symbol Device:Battery
- added C1, C2, C3, C4: C, Capacitor_SMD:C_1206_3216Metric, symbol Device:C
- added C5: C_Polarized_US, symbol Device:C_Polarized_US
- added D1, D2: LED, LED_SMD:LED_1206_3216Metric, symbol Device:LED
- added H1, H2, H3, H4: MountingHole, symbol Mechanical:MountingHole
- added R1, R2, R3, R4, R5, R6, R7: R, Resistor_SMD:R_1206_3216Metric, symbol Device:R
- added U1, U2: 24LC1025, Package_SO:SOIC-8_3.9x4.9mm_P1.27mm, symbol Memory_EEPROM:24LC1025
- added U3: DS1337S_, Real Time Clock DS1337S:SOIC127P600X175-8N, symbol Real Time Clock DS1337S:DS1337S_
- added U4: ATMEGA328P-AU, MCU_8-bit:QFP80P900X900X120-32N, symbol MCU_8-bit:ATMEGA328P-AU
- added Y1, Y2: Crystal, Crystal:Crystal_SMD_2012-2Pin_2.0x1.2mm, symbol Device:Crystal
Connections:
- new net: U4.21 (GND), U4.3 (GND), U4.5 (GND)
- new net: U4.4 (VCC), U4.6 (VCC)
Other:
- added sheet Connectors (Connectors.kicad_sch)
